File: esp32-based-motherboard.kicad_sch (KiCad schematic)
At the start: 69 parts, among them J3 USB_C_Receptacle_USB2.0_16P, J4 USB_A, J5 USB_C_Receptacle_USB2.0_16P, J6 USB_C_Receptacle_USB2.0_16P, J7 Conn_01x03_Pin, J8 Conn_01x03_Pin, SW1 SW_Push, SW2 SW_Push, SW3 SW_Push, SW4 SW_Push, SW5 SW_SPST, U12 CP2102N-Axx-xQFN24, U4 ESP32-P4_MODULE, U6 ADM3053

Commit message: Updated footprint
Parts:
- D16, D17: footprint (none) -> LED_SMD:LED_0603_1608Metric
- FB1, FB2: footprint (none) -> Inductor_SMD:L_0603_1608Metric
- J3, J5, J6: footprint (none) -> Connector_USB:USB_C_Receptacle_GCT_USB4105-xx-A_16P_TopMnt_Horizontal
- J4: footprint (none) -> Connector_USB:USB_A_Molex_67643_Horizontal
- J7, J8: footprint (none) -> Connector_PinHeader_2.54mm:PinHeader_1x03_P2.54mm_Vertical
- R10, R11, R12, R13, R14, R15, R17, R18, R19, R20, R21, R23, R24, R25, R29, R31, R4, R5, R6, R7, R8, R9: footprint (none) -> Resistor_SMD:R_0603_1608Metric
- SW5: footprint (none) -> Button_Switch_THT:SW_DIP_SPSTx01_Slide_9.78x4.72mm_W7.62mm_P2.54mm
Changed lines of the file:
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@@
 			)
 		)
-		(property "Footprint" ""
+		(property "Footprint" "LED_SMD:LED_0603_1608Metric"
 			(at 228.6 236.22 0)
 			(effects
@@
 			)
 		)
-		(property "Footprint" ""
+		(property "Footprint" "Resistor_SMD:R_0603_1608Metric"
 			(at 174.498 209.55 90)
 			(effects
@@
 			)
 		)
-		(property "Footprint" ""
+		(property "Footprint" "Resistor_SMD:R_0603_1608Metric"
 			(at 58.42 222.758 90)
 			(effects
@@
 			)
 		)
-		(property "Footprint" ""
+		(property "Footprint" "Resistor_SMD:R_0603_1608Metric"
 			(at 184.15 201.422 90)
 			(effects
@@
 			)
 		)
-		(property "Footprint" ""
+		(property "Footprint" "Resistor_SMD:R_0603_1608Metric"
 			(at 340.36 163.322 90)
 			(effects
@@
 			)
 		)
-		(property "Footprint" ""
+		(property "Footprint" "Resistor_SMD:R_0603_1608Metric"
 			(at 62.23 160.528 90)
 			(effects
@@
 			)
 		)
-		(property "Footprint" ""
+		(property "Footprint" "Connector_USB:USB_C_Receptacle_GCT_USB4105-xx-A_16P_TopMnt_Horizontal"
 			(at 121.92 218.44 0)
 			(effects
@@
 			)
 		)
-		(property "Footprint" ""
+		(property "Footprint" "Resistor_SMD:R_0603_1608Metric"
 			(at 81.28 90.678 90)
 			(effects
@@
 			)
 		)
-		(property "Footprint" ""
+		(property "Footprint" "Resistor_SMD:R_0603_1608Metric"
 			(at 57.15 81.788 90)
 			(effects
@@
 			)
 		)
-		(property "Footprint" ""
+		(property "Footprint" "Resistor_SMD:R_0603_1608Metric"
 			(at 295.402 27.94 90)
 			(effects
@@
 			)
 		)
-		(property "Footprint" ""
+		(property "Footprint" "Resistor_SMD:R_0603_1608Metric"
 			(at 137.16 212.598 90)
 			(effects
@@
 			)
 		)
-		(property "Footprint" ""
+		(property "Footprint" "LED_SMD:LED_0603_1608Metric"
 			(at 228.6 231.14 0)
 			(effects
@@
 			)
 		)
-		(property "Footprint" ""
+		(property "Footprint" "Resistor_SMD:R_0603_1608Metric"
 			(at 174.498 220.98 90)
 			(effects
@@
 			)
 		)
-		(property "Footprint" ""
+		(property "Footprint" "Resistor_SMD:R_0603_1608Metric"
 			(at 281.432 27.94 90)
 			(effects
@@
 			)
 		)
-		(property "Footprint" ""
+		(property "Footprint" "Resistor_SMD:R_0603_1608Metric"
 			(at 81.28 95.758 90)
 			(effects
@@
 			)
 		)
-		(property "Footprint" ""
+		(property "Footprint" "Inductor_SMD:L_0603_1608Metric"
 			(at 332.232 140.97 90)
 			(effects
@@
 			)
 		)
-		(property "Footprint" ""
+		(property "Footprint" "Resistor_SMD:R_0603_1608Metric"
 			(at 219.71 234.442 90)
 			(effects
@@
 			)
 		)
-		(property "Footprint" ""
+		(property "Footprint" "Button_Switch_THT:SW_DIP_SPSTx01_Slide_9.78x4.72mm_W7.62mm_P2.54mm"
 			(at 351.79 165.1 0)
 			(effects
@@
 			)
 		)
-		(property "Footprint" ""
+		(property "Footprint" "Resistor_SMD:R_0603_1608Metric"
 			(at 320.04 131.572 90)
 			(effects
@@
 			)
 		)
-		(property "Footprint" ""
+		(property "Footprint" "Resistor_SMD:R_0603_1608Metric"
 			(at 219.71 229.362 90)
 			(effects
@@
 			)
 		)
-		(property "Footprint" ""
+		(property "Footprint" "Connector_PinHeader_2.54mm:PinHeader_1x03_P2.54mm_Vertical"
 			(at 281.94 166.37 0)
 			(effects
@@
 			)
 		)
-		(property "Footprint" ""
+		(property "Footprint" "Connector_USB:USB_C_Receptacle_GCT_USB4105-xx-A_16P_TopMnt_Horizontal"
 			(at 41.91 231.14 0)
 			(effects
@@
 			)
 		)
-		(property "Footprint" ""
+		(property "Footprint" "Resistor_SMD:R_0603_1608Metric"
 			(at 268.732 27.94 90)
 			(effects
@@
 			)
 		)
-		(property "Footprint" ""
+		(property "Footprint" "Resistor_SMD:R_0603_1608Metric"
 			(at 344.932 33.02 90)
 			(effects
@@
 			)
 		)
-		(property "Footprint" ""
+		(property "Footprint" "Connector_USB:USB_C_Receptacle_GCT_USB4105-xx-A_16P_TopMnt_Horizontal"
 			(at 41.91 90.17 0)
 			(effects
@@
 			)
 		)
-		(property "Footprint" ""
+		(property "Footprint" "Inductor_SMD:L_0603_1608Metric"
 			(at 339.09 116.332 90)
 			(effects
@@
 			)
 		)
-		(property "Footprint" ""
+		(property "Footprint" "Connector_USB:USB_A_Molex_67643_Horizontal"
 			(at 35.56 157.48 0)
 			(effects
@@
 			)
 		)
-		(property "Footprint" ""
+		(property "Footprint" "Resistor_SMD:R_0603_1608Metric"
 			(at 58.42 225.298 90)
 			(effects
@@
 			)
 		)
-		(property "Footprint" ""
+		(property "Footprint" "Connector_PinHeader_2.54mm:PinHeader_1x03_P2.54mm_Vertical"
 			(at 303.53 166.37 0)
 			(effects
@@
 			)
 		)
-		(property "Footprint" ""
+		(property "Footprint" "Resistor_SMD:R_0603_1608Metric"
 			(at 62.23 157.988 90)
 			(effects
@@
 			)
 		)
-		(property "Footprint" ""
+		(property "Footprint" "Resistor_SMD:R_0603_1608Metric"
 			(at 57.15 84.328 90)
 			(effects
@@
 			)
 		)
-		(property "Footprint" ""
+		(property "Footprint" "Resistor_SMD:R_0603_1608Metric"
 			(at 328.422 33.02 90)
 			(effects
@@
 			)
 		)
-		(property "Footprint" ""
+		(property "Footprint" "Resistor_SMD:R_0603_1608Metric"
 			(at 137.16 210.058 90)
 			(effects

Commit message: Updated Footprint
Parts:
- U4: footprint ESP32-P4:XCVR_ESP32-P4_MODULE -> Custom_Footprint:ESP32-P4_MODULE

Commit message: Finalized schematics V1
Parts:
- removed U4: ESP32-P4_MODULE, Custom_Footprint:ESP32-P4_MODULE, symbol ESP32-P4_MODULE:ESP32-P4_MODULE
- added U5: ESP32-P4_MODULE, Custom_Footprint:ESP32-P4_MODULE, symbol ESP32-P4_MODULE:ESP32-P4_MODULE
- D7, D8: value SD05C-01F -> ESD7951ST5G
- J3, J5, J6: footprint Connector_USB:USB_C_Receptacle_GCT_USB4105-xx-A_16P_TopMnt_Horizontal -> Connector_USB:USB_C_Receptacle_Palconn_UTC16-G
- J7, J8: footprint Connector_PinHeader_2.54mm:PinHeader_1x03_P2.54mm_Vertical -> Connector_JST:JST_PH_B3B-PH-K_1x03_P2.00mm_Vertical
- SW5: footprint Button_Switch_THT:SW_DIP_SPSTx01_Slide_9.78x4.72mm_W7.62mm_P2.54mm -> Custom_Footprint:DSIC01LHGET_C54957
Connections:
- net +3.3V: now also U5.84 (VBAT), U5.85 (ESP_3V3), U5.86 (ESP_3V3)
- net BOOT: now also U5.62 (GPIO35/BOOT)
- net BOOT_EN: now also U5.63 (GPIO36/BOOT_EN)
- net C6_BOOT: now also U5.9 (C6_IO9/BOOT)
- net C6_BOOT_EN: now also U5.10 (C6_IO8/BOOT_EN)
- net C6_EN: now also U5.82 (GPIO54)
- net C6_UART_RX: now also U5.4 (C6_U0RXD)
- net C6_UART_TX: now also U5.5 (C6_U0TXD)
- net CAN_RX: now also U5.58 (GPIO31)
- net CAN_TX: now also U5.59 (GPIO32)
- net EN: now also U5.87 (ESP_EN)
- net GND: now also U5.1 (GND), U5.15 (GND), U5.3 (GND), U5.33 (GND), U5.40 (GND), U5.47 (GND), U5.52 (GND), U5.83 (GND)
- net PHY_MDC: now also U5.25 (GPIO10)
- net PHY_MDIO: now also U5.26 (GPIO11)
- net PHY_Reset: now also U5.27 (GPIO12)
- net RMII_CLK: now also U5.72 (GPIO44)
- net RMII_CRSDV: now also U5.73 (GPIO45)
- net RMII_RXD0: now also U5.74 (GPIO46)
- net RMII_RXD1: now also U5.75 (GPIO47)
- net RMII_RXER: now also U5.76 (GPIO48)
- net RMII_TXD0: now also U5.69 (GPIO41)
- net RMII_TXD1: now also U5.70 (GPIO42)
- net RMII_TXEN: now also U5.68 (GPIO40)
- net USB1P1_N: now also U5.50 (GPIO24/USB1P1_N0)
- net USB1P1_P: now also U5.51 (GPIO25/USB1P1_P0)
- net USB_DM: now also U5.48 (USB_DM)
- net USB_DP: now also U5.49 (USB_DP)
Other:
- moved on the sheet: C10, C19, C20, C21, C22, C23, C24, C25, C26, C28, C29, C30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

Commit message: Updated Footprint
Parts:
- renumbered C6 to C1, C21 to C10, C19 to C11, C26 to C12, C20 to C13, C22 to C14, C23 to C15, C24 to C16, C25 to C17, C7 to C2, C9 to C3, C8 to C4, C28 to C5, C29 to C6, C10 to C7, C30 to C8, C31 to C9, D10 to D1, D18 to D10, D19 to D11, D20 to D12, D16 to D13, D17 to D14, D11 to D2, D12 to D3, D7 to D4, D13 to D5, D8 to D6, D14 to D7, D9 to D8, D15 to D9, J4 to J1, J3 to J2, J5 to J3, J6 to J4, J8 to J5, J7 to J6, R8 to R1, R18 to R10, R21 to R11, R19 to R12, R20 to R13, R23 to R14, R31 to R15, R29 to R16, R10 to R17, R11 to R18, R13 to R19, R9 to R2, R24 to R20, R15 to R21, R25 to R22, R12 to R3, R14 to R4, R4 to R5, R5 to R6, R6 to R7, R7 to R8, R17 to R9, U5 to U1, U12 to U2, U6 to U3
Other:
- moved on the sheet: R7, R8

Commit message: Updated
Parts:
- added C32, C34: 10uF, Capacitor_SMD:C_0603_1608Metric, symbol Device:C_Small
- added C33, C35: 0.1uF, Capacitor_SMD:C_0603_1608Metric, symbol Device:C_Small
Connections:
- net +5V: now also C32.1, C33.1, C34.1, C35.1
- net GND: now also C32.2, C33.2, C34.2, C35.2
- net USB_A_DM renamed USB_A_N
- net USB_A_DP renamed USB_A_P
- net USB_C_DM renamed USB_C_N
- net USB_C_DP renamed USB_C_P
- net USB_DM renamed USBHS_N
- net USB_DP renamed USBHS_P
