File: esp32-based-motherboard.kicad_pcb (KiCad board)
At the start: 4 copper layers, 85.4 x 83.8 mm, 122 parts, among them J1 USB_A, J10 Conn_01x02_Pin, J11 Conn_01x02_Pin, J2 USB_C_Receptacle_USB2.0_16P, J3 USB_C_Receptacle_USB2.0_16P, J4 USB_C_Receptacle_USB2.0_16P, J5 Conn_01x03_Pin, J6 Conn_01x03_Pin, J7 RJ45_Hanrun_HR911105A_Horizon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, J8 Conn_01x02_Pin, J9 Conn_01x02_Pin, SW1 SW_Push, SW2 SW_Push, SW3 SW_Push, SW4 SW_Push, SW5 SW_SPST, U1 ESP32-P4_MODULE, U2 CP2102N-Axx-xQFN24, U3 ADM3053, U4 LAN8720A, U5 LM2596S-12, U6 LM2596S-5, U7 AMS1117-3.3, Y1 25MHz

Commit message: Updated
Routing:
- net GND: track 35.2 -> 43.5 mm
Changed lines of the file:
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@@
 	)
 	(segment
-		(start 101 84.5)
-		(end 101 82.9)
-		(width 0.25)
-		(layer "In2.Cu")
-		(net 3)
-	)
-	(segment
 		(start 84.526946 85.418114)
 		(end 84.526946 85.426946)
@@
 	)
 	(segment
+		(start 101 82.9)
+		(end 101 84.5)
+		(width 0.5)
+		(layer "In2.Cu")
+		(net 3)
+	)
+	(segment
 		(start 84.7 85.6)
 		(end 84.7 87.7)
@@
 	)
 	(segment
+		(start 72.591656 63.991656)
+		(end 76.35 67.75)
+		(width 0.3)
+		(layer "B.Cu")
+		(net 11)
+	)
+	(segment
 		(start 102.55 82.9)
 		(end 102.55 84.5)
@@
 	)
 	(segment
+		(start 76.35 67.75)
+		(end 76.8 67.75)
+		(width 0.3)
+		(layer "B.Cu")
+		(net 11)
+	)
+	(segment
+		(start 75.9 48.6)
+		(end 77.4 48.6)
+		(width 0.3)
+		(layer "B.Cu")
+		(net 11)
+	)
+	(segment
 		(start 102.174 85.426)
 		(end 102.55 85.05)
@@
 	)
 	(segment
-		(start 77.4 48.6)
-		(end 77.4 49.5)
+		(start 72.591656 62.398114)
+		(end 72.591656 63.991656)
 		(width 0.3)
-		(layer "In2.Cu")
+		(layer "B.Cu")
 		(net 11)
 	)
 	(segment
-		(start 78.278114 50.378114)
-		(end 90.051656 50.378114)
+		(start 77.4 48.6)
+		(end 79.178114 50.378114)
 		(width 0.3)
 		(layer "In2.Cu")
@@
 	)
 	(segment
-		(start 77.4 49.5)
-		(end 78.278114 50.378114)
+		(start 79.178114 50.378114)
+		(end 90.051656 50.378114)
 		(width 0.3)
 		(layer "In2.Cu")
@@
 	)
 	(segment
-		(start 90.347656 77.347656)
-		(end 88.8 75.8)
+		(start 90.347656 82.677114)
+		(end 90.347656 77.847656)
 		(width 0.3)
 		(layer "F.Cu")
@@
 	)
 	(segment
-		(start 88.8 75.8)
-		(end 86.55 75.8)
+		(start 89.906656 83.118114)
+		(end 90.347656 82.677114)
 		(width 0.3)
 		(layer "F.Cu")
@@
 	)
 	(segment
-		(start 89.906656 83.118114)
-		(end 90.347656 82.677114)
+		(start 90.347656 77.847656)
+		(end 88.3 75.8)
 		(width 0.3)
 		(layer "F.Cu")
@@
 	)
 	(segment
-		(start 90.347656 82.677114)
-		(end 90.347656 77.347656)
+		(start 88.3 75.8)
+		(end 86.55 75.8)
 		(width 0.3)
 		(layer "F.Cu")
@@
 	)
 	(zone
+		(net 0)
+		(net_name "")
+		(layer "F.Cu")
+		(hatch full 0.5)
+		(connect_pads
+			(clearance 0)
+		)
+		(min_thickness 0.25)
+		(filled_areas_thickness no)
+		(keepout
+			(tracks allowed)
+			(vias allowed)
+			(pads allowed)
+			(copperpour not_allowed)
+			(footprints allowed)
+		)
+		(placement
+			(enabled no)
+			(sheetname "/")
+		)
+		(fill
+			(thermal_gap 0.5)
+			(thermal_bridge_width 0.5)
+		)
+		(polygon
+			(pts
+				(xy 104.1 104.9) (xy 111.1 104.9) (xy 111.2 111.9) (xy 104.2 112)
+			)
+		)
+	)
+	(zone
 		(net 1)
 		(net_name "/power_system/Vcc")
@@
 	)
 	(zone
+		(net 0)
+		(net_name "")
+		(layer "F.Cu")
+		(hatch full 0.5)
+		(connect_pads
+			(clearance 0)
+		)
+		(min_thickness 0.25)
+		(filled_areas_thickness no)
+		(keepout
+			(tracks allowed)
+			(vias allowed)
+			(pads allowed)
+			(copperpour not_allowed)
+			(footprints allowed)
+		)
+		(placement
+			(enabled no)
+			(sheetname "/")
+		)
+		(fill
+			(thermal_gap 0.5)
+			(thermal_bridge_width 0.5)
+		)
+		(polygon
+			(pts
+				(xy 67.6 47.5) (xy 67.6 73.021) (xy 85.612513 73.413612) (xy 95.712901 84.4) (xy 100.8 84.4) (xy 100.8 75.382341)
+				(xy 92 66.375282) (xy 92 62.1) (xy 87.393476 56.973303) (xy 87.295792 47.595611)
+			)
+		)
+	)
+	(zone
+		(net 0)
+		(net_name "")
+		(layer "F.Cu")
+		(hatch full 0.5)
+		(connect_pads
+			(clearance 0)
+		)
+		(min_thickness 0.25)
+		(filled_areas_thickness no)
+		(keepout
+			(tracks allowed)
+			(vias allowed)
+			(pads allowed)
+			(copperpour not_allowed)
+			(footprints allowed)
+		)
+		(placement
+			(enabled no)
+			(sheetname "/")
+		)
+		(fill
+			(thermal_gap 0.5)
+			(thermal_bridge_width 0.5)
+		)
+		(polygon
+			(pts
+				(xy 133.847358 118.515038) (xy 140.847358 118.515038) (xy 140.947358 125.515038) (xy 133.947358 125.615038)
+			)
+		)
+	)
+	(zone
 		(net 11)
 		(net_name "GND")
@@
 		(net 0)
 		(net_name "")
-		(layers "F.Cu" "In1.Cu" "In2.Cu")
+		(layers "F.Cu" "B.Cu" "In1.Cu" "In2.Cu")
 		(hatch full 0.5)
 		(connect_pads
@@
 		(polygon
 			(pts
-				(xy 67.6 47.5) (xy 67.6 71.60984) (xy 84.288627 71.973596) (xy 95.712901 84.4) (xy 100.8 84.4) (xy 100.8 77.263516)
-				(xy 92 68.256457) (xy 92 62.1) (xy 87.393476 56.973303) (xy 87.295792 47.595611)
+				(xy 66.976318 43.096517) (xy 67.178384 66.233075) (xy 76 66.233075) (xy 76 65.7) (xy 83.393813 65.7)
+				(xy 85.593813 67.9) (xy 86.293813 68) (xy 86.3 65) (xy 88.4 62.9) (xy 87.5 59.5) (xy 87.487289 52.573303)
+				(xy 87.389605 43.195611)
 			)
 		)

Commit message: Updated PCB Layout
Parts:
- moved C39 0.12 mm to (76.8, 67.1)
